Commit message: update

File: urdf/google_scan/bowl.xacro (robot description, xacro)
@@ -9,5 +9,5 @@
     <origin xyz="0 0 0" rpy="0 0 0" />
     <geometry>
-      <mesh filename="package://rgbd_gazebo/meshes/Cole_Hardware_Bowl_Scirocco_YellowBlue/meshes/model.obj" scale="1.0 1.0 1.0"/>
+      <mesh filename="package://rgbd_align/meshes/Cole_Hardware_Bowl_Scirocco_YellowBlue/meshes/model.obj" scale="1.0 1.0 1.0"/>
     </geometry>
     <material name="table_material">
@@ -18,5 +18,5 @@
       <origin xyz="0 0 0" rpy="0 0 0" />
       <geometry>
-        <mesh filename="package://rgbd_gazebo/meshes/Cole_Hardware_Bowl_Scirocco_YellowBlue/meshes/model.obj" scale="1.0 1.0 1.0"/>
+        <mesh filename="package://rgbd_align/meshes/Cole_Hardware_Bowl_Scirocco_YellowBlue/meshes/model.obj" scale="1.0 1.0 1.0"/>
       </geometry>
     </collision>

File: urdf/google_scan/shoe.xacro (robot description, xacro)
@@ -9,5 +9,5 @@
     <origin xyz="0 0 0" rpy="0 0 0" />
     <geometry>
-      <mesh filename="package://rgbd_gazebo/meshes/Mens_Gold_Cup_ASV_2Eye_Boat_Shoe_in_Cognac_Leather/meshes/model.obj" scale="1.0 1.0 1.0"/>
+      <mesh filename="package://rgbd_align/meshes/Mens_Gold_Cup_ASV_2Eye_Boat_Shoe_in_Cognac_Leather/meshes/model.obj" scale="1.0 1.0 1.0"/>
     </geometry>
     <material name="table_material">
@@ -18,5 +18,5 @@
       <origin xyz="0 0 0" rpy="0 0 0" />
       <geometry>
-        <mesh filename="package://rgbd_gazebo/meshes/Mens_Gold_Cup_ASV_2Eye_Boat_Shoe_in_Cognac_Leather/meshes/model.obj" scale="1.0 1.0 1.0"/>
+        <mesh filename="package://rgbd_align/meshes/Mens_Gold_Cup_ASV_2Eye_Boat_Shoe_in_Cognac_Leather/meshes/model.obj" scale="1.0 1.0 1.0"/>
       </geometry>
     </collision>

File: urdf/realsense/_d415.urdf.xacro (robot description, xacro)
@@ -8,6 +8,6 @@
 <robot name="sensor_d415" xmlns:xacro="http://ros.org/wiki/xacro">
   <!-- Includes -->
-  <xacro:include filename="$(find rgbd_gazebo)/urdf/realsense/_materials.urdf.xacro" />
-  <xacro:include filename="$(find rgbd_gazebo)/urdf/realsense/_usb_plug.urdf.xacro" />
+  <xacro:include filename="$(find rgbd_align)/urdf/realsense/_materials.urdf.xacro" />
+  <xacro:include filename="$(find rgbd_align)/urdf/realsense/_usb_plug.urdf.xacro" />
   <xacro:macro name="sensor_d415" params="parent *origin  name:=camera  use_nominal_extrinsics:=false add_plug:=false use_mesh:=true">
     <xacro:property name="M_PI" value="3.1415926535897931" />
@@ -46,5 +46,5 @@
           <origin xyz="${d415_cam_mount_from_center_offset} ${-d415_cam_depth_py} 0" rpy="${M_PI/2} 0 ${M_PI/2}"/>
           <geometry>
-            <mesh filename="package://rgbd_gazebo/meshes/realsense/d415.stl" />
+            <mesh filename="package://rgbd_align/meshes/realsense/d415.stl" />
           </geometry>
           <material name="aluminum"/>

File: urdf/realsense/_d435.urdf.xacro (robot description, xacro)
@@ -8,6 +8,6 @@
 <robot name="sensor_d435" xmlns:xacro="http://ros.org/wiki/xacro">
   <!-- Includes -->
-  <xacro:include filename="$(find rgbd_gazebo)/urdf/realsense/_materials.urdf.xacro" />
-  <xacro:include filename="$(find rgbd_gazebo)/urdf/realsense/_usb_plug.urdf.xacro" />
+  <xacro:include filename="$(find rgbd_align)/urdf/realsense/_materials.urdf.xacro" />
+  <xacro:include filename="$(find rgbd_align)/urdf/realsense/_usb_plug.urdf.xacro" />
   <xacro:macro name="sensor_d435" params="parent *origin name:=camera use_nominal_extrinsics:=false add_plug:=false use_mesh:=true">
     <xacro:property name="M_PI" value="3.1415926535897931" />
@@ -53,5 +53,5 @@
           <origin xyz="${d435_zero_depth_to_glass + d435_glass_to_front} ${-d435_cam_depth_py} 0" rpy="${M_PI/2} 0 ${M_PI/2}"/>
           <geometry>
-            <mesh filename="package://rgbd_gazebo/meshes/realsense/d435.dae" />
+            <mesh filename="package://rgbd_align/meshes/realsense/d435.dae" />
           </geometry>
         </xacro:if>

File: urdf/realsense/_d435i.urdf.xacro (robot description, xacro)
@@ -7,6 +7,6 @@
 -->
 <robot name="sensor_d435i" xmlns:xacro="http://ros.org/wiki/xacro">
-  <xacro:include filename="$(find rgbd_gazebo)/urdf/realsense/_d435.urdf.xacro"/>
-  <xacro:include filename="$(find rgbd_gazebo)/urdf/realsense/_d435i_imu_modules.urdf.xacro"/>
+  <xacro:include filename="$(find rgbd_align)/urdf/realsense/_d435.urdf.xacro"/>
+  <xacro:include filename="$(find rgbd_align)/urdf/realsense/_d435i_imu_modules.urdf.xacro"/>
   <xacro:macro name="sensor_d435i" params="parent *origin name:=camera use_nominal_extrinsics:=false">
     <xacro:sensor_d435 parent="${parent}" name="${name}" use_nominal_extrinsics="${use_nominal_extrinsics}">

File: urdf/realsense/_d455.urdf.xacro (robot description, xacro)
@@ -8,6 +8,6 @@
 <robot name="sensor_d455" xmlns:xacro="http://ros.org/wiki/xacro">
   <!-- Includes -->
-  <xacro:include filename="$(find rgbd_gazebo)/urdf/realsense/_materials.urdf.xacro" />
-  <xacro:include filename="$(find rgbd_gazebo)/urdf/realsense/_usb_plug.urdf.xacro" />
+  <xacro:include filename="$(find rgbd_align)/urdf/realsense/_materials.urdf.xacro" />
+  <xacro:include filename="$(find rgbd_align)/urdf/realsense/_usb_plug.urdf.xacro" />
   <xacro:macro name="sensor_d455" params="parent *origin name:=camera use_nominal_extrinsics:=false">
     <xacro:arg name="add_plug" default="false" />
@@ -55,5 +55,5 @@
         <geometry>
           <!-- <box size="${d455_cam_depth} ${d455_cam_width} ${d455_cam_height}"/> -->
-	        <mesh filename="package://rgbd_gazebo/meshes/realsense/d455.stl" scale="0.001 0.001 0.001" />
+	        <mesh filename="package://rgbd_align/meshes/realsense/d455.stl" scale="0.001 0.001 0.001" />
         </geometry>
         <material name="aluminum"/>

File: urdf/realsense/_l515.urdf.xacro (robot description, xacro)
@@ -8,6 +8,6 @@
 <robot name="sensor_l515" xmlns:xacro="http://ros.org/wiki/xacro">
   <!-- Includes -->
-  <xacro:include filename="$(find rgbd_gazebo)/urdf/realsense/_materials.urdf.xacro" />
-  <xacro:include filename="$(find rgbd_gazebo)/urdf/realsense/_usb_plug.urdf.xacro" /> <!-- this specific plug does not apply to L515 -->
+  <xacro:include filename="$(find rgbd_align)/urdf/realsense/_materials.urdf.xacro" />
+  <xacro:include filename="$(find rgbd_align)/urdf/realsense/_usb_plug.urdf.xacro" /> <!-- this specific plug does not apply to L515 -->
   <xacro:macro name="sensor_l515" params="parent *origin name:=camera use_nominal_extrinsics:=false add_plug:=false use_mesh:=true">
     <xacro:property name="M_PI" value="3.1415926535897931" />
@@ -63,5 +63,5 @@
           <origin xyz="${l515_zero_depth_to_glass} 0 ${-l515_cam_center_to_depth_pz}" rpy="${M_PI/2} 0 ${M_PI/2}"/>
           <geometry>
-              <mesh filename="package://rgbd_gazebo/meshes/realsense/l515.dae" />
+              <mesh filename="package://rgbd_align/meshes/realsense/l515.dae" />
           </geometry>
         </xacro:if>

File: urdf/realsense/_r410.urdf.xacro (robot description, xacro)
@@ -8,5 +8,5 @@
 <robot name="sensor_r410" xmlns:xacro="http://ros.org/wiki/xacro">
   <!-- Includes -->
-  <xacro:include filename="$(find rgbd_gazebo)/urdf/realsense/_materials.urdf.xacro" />
+  <xacro:include filename="$(find rgbd_align)/urdf/realsense/_materials.urdf.xacro" />
   <xacro:macro name="sensor_r410" params="parent *origin  name:=camera  use_nominal_extrinsics:=false">
     <xacro:property name="M_PI" value="3.1415926535897931" />
@@ -38,5 +38,5 @@
         <geometry>
           <box size="${r410_cam_width} ${r410_cam_height} ${r410_cam_depth}"/>
-          <!--<mesh filename="package://rgbd_gazebo/meshes/realsense/r410/r410.dae" />-->
+          <!--<mesh filename="package://rgbd_align/meshes/realsense/r410/r410.dae" />-->
         </geometry>
         <material name="aluminum"/>

File: urdf/realsense/_r430.urdf.xacro (robot description, xacro)
@@ -8,5 +8,5 @@
 <robot name="sensor_r430" xmlns:xacro="http://ros.org/wiki/xacro">
   <!-- Includes -->
-  <xacro:include filename="$(find rgbd_gazebo)/urdf/realsense/_materials.urdf.xacro" />
+  <xacro:include filename="$(find rgbd_align)/urdf/realsense/_materials.urdf.xacro" />
   <xacro:macro name="sensor_r430" params="parent *origin name:=camera use_nominal_extrinsics:=false">
   <xacro:property name="M_PI" value="3.1415926535897931" />
@@ -39,5 +39,5 @@
         <geometry>
           <box size="${r430_cam_width} ${r430_cam_height} ${r430_cam_depth}"/>
-          <!--<mesh filename="package://rgbd_gazebo/meshes/realsense/r430/r430.dae" />-->
+          <!--<mesh filename="package://rgbd_align/meshes/realsense/r430/r430.dae" />-->
         </geometry>
         <material name="aluminum"/>

File: urdf/realsense/_usb_plug.urdf.xacro (robot description, xacro)
@@ -20,5 +20,5 @@
         <geometry>
           <!--box size="0.044850 0.008 0.0185" /-->
-          <mesh filename="package://rgbd_gazebo/meshes/realsense/plug.stl" />
+          <mesh filename="package://rgbd_align/meshes/realsense/plug.stl" />
         </geometry>
         <material name="plastic"/>
@@ -28,5 +28,5 @@
         <geometry>
           <!--box size="0.044850 0.008 0.0185" /-->
-          <mesh filename="package://rgbd_gazebo/meshes/realsense/plug_collision.stl" />
+          <mesh filename="package://rgbd_align/meshes/realsense/plug_collision.stl" />
         </geometry>
       </collision>

File: urdf/realsense/d435_gazebo.xacro (robot description, xacro)
@@ -1,8 +1,8 @@
 <?xml version="1.0"?>
 <robot name="realsense2_camera" xmlns:xacro="http://ros.org/wiki/xacro">
-  <xacro:arg name="use_nominal_extrinsics" default="false"/>
+  <xacro:arg name="use_nominal_extrinsics" default="true"/>
   <xacro:arg name="add_plug" default="false" />
   <xacro:arg name="use_mesh" default="true" />
-  <xacro:include filename="$(find rgbd_gazebo)/urdf/realsense/_d435.urdf.xacro" />
+  <xacro:include filename="$(find rgbd_align)/urdf/realsense/_d435.urdf.xacro" />
   <link name="d435_base" />
   <xacro:sensor_d435 parent="d435_base" use_nominal_extrinsics="$(arg use_nominal_extrinsics)" add_plug="$(arg add_plug)" use_mesh="$(arg use_mesh)">

File: urdf/realsense/test_d415_camera.urdf.xacro (robot description, xacro)
@@ -4,5 +4,5 @@
   <xacro:arg name="add_plug" default="false" />
   <xacro:arg name="use_mesh" default="true" />
-  <xacro:include filename="$(find rgbd_gazebo)/urdf/realsense/_d415.urdf.xacro" />
+  <xacro:include filename="$(find rgbd_align)/urdf/realsense/_d415.urdf.xacro" />
   <link name="base_link" />
   <xacro:sensor_d415 parent="base_link" use_nominal_extrinsics="$(arg use_nominal_extrinsics)" add_plug="$(arg add_plug)" use_mesh="$(arg use_mesh)">

File: urdf/realsense/test_d435_camera.urdf.xacro (robot description, xacro)
@@ -4,5 +4,5 @@
   <xacro:arg name="add_plug" default="false" />
   <xacro:arg name="use_mesh" default="true" />
-  <xacro:include filename="$(find rgbd_gazebo)/urdf/realsense/_d435.urdf.xacro" />
+  <xacro:include filename="$(find rgbd_align)/urdf/realsense/_d435.urdf.xacro" />
   <link name="base_link" />
   <xacro:sensor_d435 parent="base_link" use_nominal_extrinsics="$(arg use_nominal_extrinsics)" add_plug="$(arg add_plug)" use_mesh="$(arg use_mesh)">

File: urdf/realsense/test_d435_multiple_cameras.urdf.xacro (robot description, xacro)
@@ -2,5 +2,5 @@
 <robot name="realsense2_camera" xmlns:xacro="http://ros.org/wiki/xacro">
   <xacro:arg name="use_nominal_extrinsics" default="false"/>
-  <xacro:include filename="$(find rgbd_gazebo)/urdf/realsense/_d435.urdf.xacro" />
+  <xacro:include filename="$(find rgbd_align)/urdf/realsense/_d435.urdf.xacro" />
   <link name="base_link" />
   <xacro:sensor_d435 parent="base_link" name="camera1" use_nominal_extrinsics="$(arg use_nominal_extrinsics)">

File: urdf/realsense/test_d435i_camera.urdf.xacro (robot description, xacro)
@@ -2,5 +2,5 @@
 <robot name="realsense2_camera" xmlns:xacro="http://www.ros.org/wiki/xacro">
   <xacro:arg name="use_nominal_extrinsics" default="false" />
-  <xacro:include filename="$(find rgbd_gazebo)/urdf/realsense/_d435i.urdf.xacro"/>
+  <xacro:include filename="$(find rgbd_align)/urdf/realsense/_d435i.urdf.xacro"/>
   <link name="base_link" />
   <xacro:sensor_d435i parent="base_link" use_nominal_extrinsics="$(arg use_nominal_extrinsics)">

File: urdf/realsense/test_d455_camera.urdf.xacro (robot description, xacro)
@@ -2,5 +2,5 @@
 <robot name="realsense2_camera" xmlns:xacro="http://ros.org/wiki/xacro">
   <xacro:arg name="use_nominal_extrinsics" default="false"/>
-  <xacro:include filename="$(find rgbd_gazebo)/urdf/realsense/_d455.urdf.xacro" />
+  <xacro:include filename="$(find rgbd_align)/urdf/realsense/_d455.urdf.xacro" />
   <link name="base_link" />
   <xacro:sensor_d455 parent="base_link" use_nominal_extrinsics="$(arg use_nominal_extrinsics)">

File: urdf/realsense/test_l515_camera.urdf.xacro (robot description, xacro)
@@ -4,5 +4,5 @@
   <xacro:arg name="add_plug" default="false" />
   <xacro:arg name="use_mesh" default="true" />
-  <xacro:include filename="$(find rgbd_gazebo)/urdf/realsense/_l515.urdf.xacro" />
+  <xacro:include filename="$(find rgbd_align)/urdf/realsense/_l515.urdf.xacro" />
   <link name="base_link" />
   <xacro:sensor_l515 parent="base_link" use_nominal_extrinsics="$(arg use_nominal_extrinsics)" add_plug="$(arg add_plug)" use_mesh="$(arg use_mesh)">

File: urdf/realsense/test_r410_camera.urdf.xacro (robot description, xacro)
@@ -2,5 +2,5 @@
 <robot name="realsense2_camera" xmlns:xacro="http://ros.org/wiki/xacro">
   <xacro:arg name="use_nominal_extrinsics" default="false"/>
-  <xacro:include filename="$(find rgbd_gazebo)/urdf/realsense/_r410.urdf.xacro" />
+  <xacro:include filename="$(find rgbd_align)/urdf/realsense/_r410.urdf.xacro" />
   <link name="base_link" />
   <xacro:sensor_r410 parent="base_link" use_nominal_extrinsics="$(arg use_nominal_extrinsics)">

File: urdf/realsense/test_r430_camera.urdf.xacro (robot description, xacro)
@@ -2,5 +2,5 @@
 <robot name="realsense2_camera" xmlns:xacro="http://ros.org/wiki/xacro">
   <xacro:arg name="use_nominal_extrinsics" default="false"/>
-  <xacro:include filename="$(find rgbd_gazebo)/urdf/realsense/_r430.urdf.xacro" />
+  <xacro:include filename="$(find rgbd_align)/urdf/realsense/_r430.urdf.xacro" />
   <link name="base_link" />
   <xacro:sensor_r430 parent="base_link" use_nominal_extrinsics="$(arg use_nominal_extrinsics)">
